File: Scanner/HR_SR04_Multiplex_Shield/HC_SR04_Multiplex_Shield.sch (KiCad schematic (older format))
At the start: 21 parts, among them J1 Conn_01x02, J10 Conn_01x02, J11 Conn_01x02, J2 Conn_01x02, J3 Conn_01x02, J4 Conn_01x02, J5 Conn_01x02, J6 Conn_01x02, J7 Conn_01x02, J8 Conn_01x02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

Commit message: routed and ready for manufacture
Connections:
- net 12(MISO) is gone; now on net 12: P3.6 (Pin_6)
- net 3(**) is gone; now on net 3: P4.5 (Pin_5)
- net 5(**) is gone; now on net 5: P4.3 (Pin_3)
- net 6 is gone; now on net 2: U1.10 (S0)
- net 9 is gone; now on net 5: U1.13 (S3)
- net 3: now also U1.11 (S1)
- net 4: now also U1.14 (S2)
- net 7: no longer U1.11 (S1)
- net 8: no longer U1.14 (S2)
- net A4(SDA): no longer P3.2 (Pin_2)
- net A5(SCL): no longer P3.1 (Pin_1)
- new net A4: P3.2 (Pin_2)
- new net A5: P3.1 (Pin_1)
Changed lines of the file:
@@
 EESchema Schematic File Version 4
-LIBS:OrangePipShield-cache
+LIBS:HC_SR04_Multiplex_Shield-cache
 EELAYER 30 0
 EELAYER END
@@
 1(Tx)
 Text Label 5100 4000 0    60   ~ 0
-3(**)
+3
 Text Label 5100 3900 0    60   ~ 0
 4
 Text Label 5100 3800 0    60   ~ 0
-5(**)
+5
 Text Label 5100 3700 0    60   ~ 0
 6(**)
@@
 11(TRIG)
 Text Label 5100 3000 0    60   ~ 0
-12(MISO)
+12
 Text Label 5100 2900 0    60   ~ 0
 13(SCK)
@@
 NoConn ~ 3950 2900
 Text Label 5100 2600 0    60   ~ 0
-A4(SDA)
+A4
 Text Label 5100 2500 0    60   ~ 0
-A5(SCL)
+A5
 Text Notes 4050 1775 0    60   ~ 0
 Holes
@@
 5
 Text Label 6250 2200 0    50   ~ 0
-6
+2
 Text Label 6250 2300 0    50   ~ 0
-7
+3
 Text Label 6250 2400 0    50   ~ 0
-8
+4
 Text Label 6250 2500 0    50   ~ 0
-9
+5
 Text Label 6275 2900 2    50   ~ 0
 12
