File: Mask/Alexa_kicad_PCB/Alexa_kicad_PCB.sch (KiCad schematic (older format))
At the start: 9 parts

Commit message: schematic progressed 20% completed
Parts:
- added C?: 10uF, symbol Device:C_Small
- added C? (x2): 10p, symbol Device:C_Small
- added J?: Jack-DC, symbol Connector:Jack-DC
- added R? (x5): 100k, symbol Device:R_Small
- added U?: LM1117-3.3, symbol Regulator_Linear:LM1117-3.3
- added Y?: 12Mhz, symbol Device:Crystal
Connections:
- net +3V3: now also R?.1, R?.1, R?.1, U?.2 (VO)
- net GND: now also C?.2, C?.2, C?.2, J?.2, R?.1, R?.1, U?.1 (GND)
- net at U?.28 (PB2): now also R?.2
- net at U?.30 (PB11): now also R?.2
- net at U?.43 (PA10): now also R?.2
- net at U?.5 (PH0): now also C?.1, Y?.1
- net at U?.52 (PC11): now also R?.2
- net at U?.57 (PB5): now also R?.2
- net at U?.6 (PH1): now also C?.1, Y?.2
- new net +5V: C?.1, J?.1, U?.3 (VI)
Other:
- moved on the sheet: C?

Commit message: started audio section of schematic
Parts:
- added J?: Audio In, symbol Connector:AudioJack2_Ground
- added J?: Audio Out, symbol Connector:AudioJack2_Ground
- added U?: OPAMP, symbol pspice:OPAMP
Connections:
- new net: J?.S, J?.S
- new net: J?.T, J?.T
Changed lines of the file:
@@
 Wire Wire Line
 	6200 4150 6200 4200
+$Comp
+L Connector:AudioJack2_Ground J?
+U 1 1 5F09035A
+P 1000 6650
+F 0 "J?" H 1032 6975 50  0000 C CNN
+F 1 "Audio In" H 1032 6884 50  0000 C CNN
+F 2 "" H 1000 6650 50  0001 C CNN
+F 3 "~" H 1000 6650 50  0001 C CNN
+	1    1000 6650
+	1    0    0    -1
+$EndComp
+$Comp
+L Connector:AudioJack2_Ground J?
+U 1 1 5F094637
+P 1000 7350
+F 0 "J?" H 1032 7675 50  0000 C CNN
+F 1 "Audio Out" H 1032 7584 50  0000 C CNN
+F 2 "" H 1000 7350 50  0001 C CNN
+F 3 "~" H 1000 7350 50  0001 C CNN
+	1    1000 7350
+	1    0    0    -1
+$EndComp
+Wire Wire Line
+	1200 6550 1350 6550
+Wire Wire Line
+	1350 6550 1350 7250
+Wire Wire Line
+	1350 7250 1200 7250
+Wire Wire Line
+	1200 6650 1400 6650
+Wire Wire Line
+	1400 6650 1400 7350
+Wire Wire Line
+	1400 7350 1200 7350
+$Comp
+L pspice:OPAMP U?
+U 1 1 5F0A6325
+P 2450 6850
+F 0 "U?" H 2794 6896 50  0000 L CNN
+F 1 "OPAMP" H 2794 6805 50  0000 L CNN
+F 2 "" H 2450 6850 50  0001 C CNN
+F 3 "~" H 2450 6850 50  0001 C CNN
+	1    2450 6850
+	1    0    0    -1
+$EndComp
 $EndSCHEMATC
