File: Mask/Alexa_kicad_PCB/_autosave-Alexa_kicad_PCB.sch (KiCad schematic (older format))
At the start: 28 parts

Commit message: finished analog schematic layout part
Connections:
- net +5V: now also M?.2 (+), M?.2 (+), M?.2 (+)
- net GND: now also M?.3 (-), M?.3 (-), M?.3 (-)
Other:
- moved on the sheet: C?, D?, J?, M?, R?, U?
