File: Mask/Alexa_kicad_PCB/Alexa_kicad_PCB.kicad_pcb (KiCad board)
At the start: 2 copper layers, 28 parts, among them J1 Jack-DC, J2 USB_B_Micro, M1 Motor_Servo, M2 Motor_Servo, M3 Motor_Servo, U1 TLV2372, U2 LM1117-3.3, U3 STM32F405RGTx, X1 1503_09, X2 1503_09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

Commit message: footprints placed, ready for routing
Parts:
- added REF**: MountingHole_3.2mm_M3, MountingHole:MountingHole_3.2mm_M3, F.Cu at (101.6, 73.7)
- added REF**: MountingHole_3.2mm_M3, MountingHole:MountingHole_3.2mm_M3, F.Cu at (144.8, 109.2)
- moved J1 34.3 mm to (139.7, 85.1), turned to 90 degrees
- moved U2 30.6 mm to (106.7, 99.1)
- moved R4 26.0 mm to (100.0, 94.0)
- moved C2 25.9 mm to (100.7, 85.9)
- moved R6 25.9 mm to (100.7, 88.8)
- moved R7 25.9 mm to (105.2, 85.9)
- moved C3 13.7 mm to (117.4, 103.2)
- moved R2 13.7 mm to (117.4, 106.1)
- moved R10 13.7 mm to (121.8, 106.8)
- moved R5 13.7 mm to (121.8, 103.8)
- moved R9 10.8 mm to (128.6, 104.1)
- moved M1 7.62 mm to (137.4, 111.3)
- moved M2 7.62 mm to (113.5, 111.5)
- moved M3 7.62 mm to (125.7, 111.5)
- moved U3 5.57 mm to (124.5, 94.0), turned to 45 degrees
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Routing:
- added copper zone on F.Cu, net GND
Other:
- board outline added: 53.3 x 45.7 mm

Commit message: routing completed
Parts:
- added D2: BAR43FILM, Package_TO_SOT_SMD:SOT-23, F.Cu at (135.4, 85.1)
- added J3: Conn_01x07_Male, Connector_PinHeader_2.54mm:PinHeader_1x07_P2.54mm_Horizontal, F.Cu at (148.6, 89.4)
- moved D1 36.6 mm to (103.4, 82.7), turned to 90 degrees
- moved R6 28.9 mm to (125.8, 103.3)
- moved C1 28.0 mm to (113.5, 87.4), turned to 180 degrees
- moved R1 24.2 mm to (108.6, 84.2)
- moved C3 22.8 mm to (100.4, 87.9)
- moved R2 21.9 mm to (113.6, 84.6)
- moved R10 21.0 mm to (135.0, 90.4)
- moved R3 20.4 mm to (127.0, 84.8)
- moved R5 20.3 mm to (130.6, 85.5), turned to 270 degrees
- moved R7 17.7 mm to (122.9, 85.0)
- moved C2 15.7 mm to (98.8, 101.5), turned to 90 degrees
- moved R9 12.8 mm to (134.9, 93.0)
- moved Y1 10.3 mm to (114.6, 93.2)
- moved C5 8.99 mm to (113.5, 103.6)
- moved C6 8.84 mm to (113.5, 106.2)
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Connections:
- net Net-(U3-Pad38) renamed /38_BO
- net Net-(U3-Pad39) renamed /39_BO
- net Net-(U3-Pad40) renamed /40_BO
- net Net-(U3-Pad41) renamed /41_BO
- net Net-(U3-Pad42) renamed /42_BO
- J2 pad 5: Net-(J2-Pad5) -> GND
- J2 pad 6: Net-(J2-Pad6) -> GND
- U3 pad 33: Net-(U3-Pad33) -> /33_BO
- U3 pad 34: Net-(U3-Pad34) -> /34_BO
- U3 pad 35: Net-(U3-Pad35) -> /35_BO
- U3 pad 36: Net-(U3-Pad36) -> /36_BO
- U3 pad 37: Net-(U3-Pad37) -> /37_BO
Routing:
- net +5V: track 0.00 -> 129.5 mm, vias 0 -> 2
- net +3V3: track 0.00 -> 115.0 mm
- net Net-(U1-Pad3): track 0.00 -> 49.5 mm
- net /EYES_SERVO: track 0.00 -> 29.0 mm
- net Net-(J2-Pad3): track 0.00 -> 28.1 mm
- net Net-(J2-Pad2): track 0.00 -> 24.4 mm
- net /37_BO: track 0.00 -> 21.1 mm
- net /36_BO: track 0.00 -> 20.2 mm
- net /33_BO: track 0.00 -> 19.4 mm
- net /35_BO: track 0.00 -> 19.4 mm
- net /34_BO: track 0.00 -> 18.8 mm
- net Net-(D2-Pad1): track 0.00 -> 18.1 mm
- net Net-(D1-Pad1): track 0.00 -> 18.1 mm
- net /MOUTH_SERVO: track 0.00 -> 17.2 mm
- net /NECK_SERVO: track 0.00 -> 17.1 mm
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Other:
- rule trace_min: 0.2 -> 0.1
- rule via_min_drill: 0.3 -> 0.2

Commit message: silkscreen text partially finished
Other:
- board text added: "EYES"
- board text added: "MOUTH"
- board text added: "NECK"
- board text added: "Spooky Alexa"
- board text added: "v0.1"
- board text added: "wattnotions.com/sa"
Changed lines of the file:
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@@
   (general
     (thickness 1.6)
-    (drawings 8)
+    (drawings 14)
     (tracks 214)
     (zones 0)
@@
     (tags capacitor)
     (attr smd)
-    (fp_text reference C6 (at 0 -1.65) (layer F.SilkS)
+    (fp_text reference C6 (at 2.906 0.127) (layer F.SilkS)
       (effects (font (size 1 1) (thickness 0.15)))
     )
@@
     (tags resistor)
     (attr smd)
-    (fp_text reference R9 (at 0 -1.65) (layer F.SilkS)
+    (fp_text reference R9 (at 0.0635 1.8415) (layer F.SilkS)
       (effects (font (size 1 1) (thickness 0.15)))
     )
@@
     )
   )
+  (gr_text v0.1 (at 141.1605 98.9965 45) (layer F.SilkS)
+    (effects (font (size 1.2 1.2) (thickness 0.2)))
+  )
+  (gr_text wattnotions.com/sa (at 139.6365 97.155 45) (layer F.SilkS)
+    (effects (font (size 1.2 1.2) (thickness 0.2)))
+  )
+  (gr_text "Spooky Alexa" (at 137.2235 95.631 45) (layer F.SilkS)
+    (effects (font (size 1.5 1.5) (thickness 0.3) italic))
+  )
+  (gr_text EYES (at 134.874 108.966) (layer F.SilkS)
+    (effects (font (size 1.5 1.5) (thickness 0.3)))
+  )
+  (gr_text NECK (at 123.1265 109.093) (layer F.SilkS)
+    (effects (font (size 1.5 1.5) (thickness 0.3)))
+  )
+  (gr_text MOUTH (at 110.6805 109.22) (layer F.SilkS)
+    (effects (font (size 1.5 1.5) (thickness 0.3)))
+  )
   (gr_line (start 99.06 68.58) (end 147.32 68.58) (layer Edge.Cuts) (width 0.05))

Commit message: silk screen done, board finished
Other:
- board text added: "3V3"
- board text added: "B12"
- board text added: "B13"
- board text added: "B14"
- board text added: "B15"
- board text added: "C6"
- board text added: "GND"
Changed lines of the file:
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@@
   (general
     (thickness 1.6)
-    (drawings 14)
+    (drawings 23)
     (tracks 214)
     (zones 0)
@@
   )
   (setup
-    (last_trace_width 0.15)
+    (last_trace_width 0.25)
     (user_trace_width 0.1)
     (user_trace_width 0.15)
@@
     (tags "mounting hole 3.2mm no annular m3")
     (attr virtual)
-    (fp_text reference REF** (at 0 -4.2) (layer F.SilkS)
+    (fp_text reference REF** (at 0 -4.2) (layer F.SilkS) hide
       (effects (font (size 1 1) (thickness 0.15)))
     )
@@
     (tags "mounting hole 3.2mm no annular m3")
     (attr virtual)
-    (fp_text reference REF** (at 0 -4.2) (layer F.SilkS)
+    (fp_text reference REF** (at -4.064 -3.048) (layer F.SilkS) hide
       (effects (font (size 1 1) (thickness 0.15)))
     )
@@
     )
   )
-  (gr_text v0.1 (at 141.1605 98.9965 45) (layer F.SilkS)
-    (effects (font (size 1.2 1.2) (thickness 0.2)))
-  )
-  (gr_text wattnotions.com/sa (at 139.6365 97.155 45) (layer F.SilkS)
-    (effects (font (size 1.2 1.2) (thickness 0.2)))
+  (gr_circle (center 110.236 86.106) (end 110.236 86.36) (layer F.SilkS) (width 0.12))
+  (gr_circle (center 118.11 88.138) (end 118.364 88.392) (layer F.SilkS) (width 0.12))
+  (gr_text 3V3 (at 145.542 104.648) (layer F.SilkS)
+    (effects (font (size 1 1) (thickness 0.2)))
+  )
+  (gr_text GND (at 145.542 102.108) (layer F.SilkS)
+    (effects (font (size 1 1) (thickness 0.2)))
+  )
+  (gr_text B12 (at 145.542 99.568) (layer F.SilkS)
+    (effects (font (size 1 1) (thickness 0.2)))
+  )
+  (gr_text B13 (at 145.542 97.028) (layer F.SilkS)
+    (effects (font (size 1 1) (thickness 0.2)))
+  )
+  (gr_text B14 (at 145.542 94.488) (layer F.SilkS)
+    (effects (font (size 1 1) (thickness 0.2)))
+  )
+  (gr_text B15 (at 145.542 91.948) (layer F.SilkS)
+    (effects (font (size 1 1) (thickness 0.2)))
+  )
+  (gr_text C6 (at 146.05 89.408) (layer F.SilkS)
+    (effects (font (size 1 1) (thickness 0.2)))
+  )
+  (gr_text v0.1 (at 140.208 98.298 45) (layer F.SilkS)
+    (effects (font (size 1 1) (thickness 0.2)))
+  )
+  (gr_text wattnotions.com/sa (at 138.684 97.282 45) (layer F.SilkS)
+    (effects (font (size 0.8 0.8) (thickness 0.2)))
   )
   (gr_text "Spooky Alexa" (at 137.2235 95.631 45) (layer F.SilkS)

Commit message: v0.2 routing started
Parts:
- removed REF** (x2): MountingHole_3.2mm_M3, MountingHole:MountingHole_3.2mm_M3
- added C7: 2.2uF, Capacitor_SMD:C_0603_1608Metric, F.Cu at (128.5, 105.5)
- added C8: 2.2uF, Capacitor_SMD:C_0603_1608Metric, F.Cu at (178.2, 74.1)
- added D3: LED, LED_SMD:LED_0603_1608Metric, F.Cu at (138.6, 100.1)
- added D4: LED, LED_SMD:LED_0603_1608Metric, F.Cu at (138.6, 105.7)
- added D5: LED, LED_SMD:LED_0603_1608Metric, F.Cu at (138.6, 103.8)
- added D6: LED, LED_SMD:LED_0603_1608Metric, F.Cu at (138.6, 101.9)
- added D7: LED, LED_SMD:LED_0603_1608Metric, F.Cu at (188.1, 67.2)
- added R11: 10K, Resistor_SMD:R_0603_1608Metric, F.Cu at (146.4, 120.6)
- added R12: 100K, Resistor_SMD:R_0603_1608Metric, F.Cu at (126.9, 84.8)
- added R13: 4K7, Resistor_SMD:R_0603_1608Metric, F.Cu at (130.7, 103.2)
- added R14: R_Small, Resistor_SMD:R_0603_1608Metric, F.Cu at (190.3, 73.0)
- added R15: 100K, Resistor_SMD:R_0603_1608Metric, F.Cu at (194.3, 70.5)
- added R16: 100K, Resistor_SMD:R_0603_1608Metric, F.Cu at (129.9, 86.2)
- added R17: 100K, Resistor_SMD:R_0603_1608Metric, F.Cu at (125.9, 103.4)
- added R18: 100K, Resistor_SMD:R_0603_1608Metric, F.Cu at (122.8, 85.1)
- added SW1: SW_Push, Button_Switch_SMD:SW_SPST_B3U-1000P, F.Cu at (179.4, 82.7)
- added SW2: SW_Push, Button_Switch_SMD:SW_SPST_B3U-1000P, F.Cu at (179.1, 68.1)
- added SW3: SW_Push, Button_Switch_SMD:SW_SPST_B3U-1000P, F.Cu at (158.8, 114.9)
- C1, C2, C3, C4, C5, C6: footprint Capacitor_SMD:C_0805_2012Metric -> Capacitor_SMD:C_0603_1608Metric
- R1, R10, R2, R4, R9: footprint Resistor_SMD:R_0805_2012Metric -> Resistor_SMD:R_0603_1608Metric
- R3, R5, R6, R7: value 100k -> 560R; footprint Resistor_SMD:R_0805_2012Metric -> Resistor_SMD:R_0603_1608Metric
- R8: value 100k -> 4K7; footprint Resistor_SMD:R_0805_2012Metric -> Resistor_SMD:R_0603_1608Metric
- moved R8 75.0 mm to (194.0, 62.9), turned to 0 degrees
- moved R7 21.0 mm to (135.2, 101.9), turned to 180 degrees
- moved R5 20.8 mm to (135.2, 105.8), turned to 180 degrees
- moved R3 17.4 mm to (135.2, 100.1), turned to 180 degrees
- moved R6 9.41 mm to (135.2, 103.6), turned to 180 degrees
Connections:
- net Net-(U3-Pad55) renamed /PB3-USR_SW
- R3 pad 1: +3V3 -> Net-(D3-Pad2)
- R3 pad 2: Net-(R3-Pad2) -> /PA13-RED
- R5 pad 1: +3V3 -> Net-(D4-Pad2)
- R5 pad 2: Net-(R5-Pad2) -> /PA14-GRN
- R6 pad 1: GND -> Net-(D5-Pad2)
- R6 pad 2: Net-(R6-Pad2) -> /PA15-YEL
- R7 pad 1: GND -> Net-(D6-Pad2)
- R7 pad 2: Net-(R7-Pad2) -> /PB4-BLU
- R8 pad 1: +3V3 -> /NRST
- R8 pad 2: Net-(R8-Pad2) -> +3V3
- U3 pad 28: Net-(R6-Pad2) -> /PB2-(DFU)
- U3 pad 30: Net-(R8-Pad2) -> /PB11-(DFU)
- U3 pad 43: Net-(R5-Pad2) -> /PA10-(DFU)
- U3 pad 46: Net-(U3-Pad46) -> /PA13-RED
- U3 pad 49: Net-(U3-Pad49) -> /PA14-GRN
- U3 pad 50: Net-(U3-Pad50) -> /PA15-YEL
- U3 pad 52: Net-(R3-Pad2) -> /PC11-(DFU)
- U3 pad 56: Net-(U3-Pad56) -> /PB4-BLU
- U3 pad 57: Net-(R7-Pad2) -> /PB5-(DFU)
- U3 pad 60: Net-(U3-Pad60) -> /BOOT0-(DFU)
- U3 pad 7: Net-(U3-Pad7) -> /NRST
Routing:
- net Net-(R5-Pad2): track 8.67 -> 0.00 mm
- net /PA10-(DFU): track 0.00 -> 8.67 mm
- net Net-(R8-Pad2): track 4.95 -> 0.00 mm
- net /PB11-(DFU): track 0.00 -> 4.95 mm
- net Net-(R3-Pad2): track 3.96 -> 0.00 mm
- net /PC11-(DFU): track 0.00 -> 3.96 mm
- net Net-(R6-Pad2): track 3.82 -> 0.00 mm
- net /PB2-(DFU): track 0.00 -> 3.82 mm
- net Net-(R7-Pad2): track 3.57 -> 0.00 mm
- net /PB5-(DFU): track 0.00 -> 3.57 mm
Other:
- board text removed: "Spooky Alexa"
- board text removed: "v0.1"
- board text removed: "wattnotions.com/sa"

Commit message: v0.2 routing completed
Parts:
- added REF**: MountingHole_3mm_Pad, MountingHole:MountingHole_3mm_Pad, F.Cu at (102.4, 73.8)
- added REF**: MountingHole_3mm_Pad, MountingHole:MountingHole_3mm_Pad, F.Cu at (144.4, 110.4)
- moved R14 90.0 mm to (103.3, 95.8), turned to 180 degrees
- moved D7 86.3 mm to (106.7, 95.8)
- moved SW1 82.8 mm to (101.5, 110.7), turned to 180 degrees
- moved R8 80.8 mm to (117.0, 87.4), turned to 180 degrees
- moved R15 74.2 mm to (121.6, 85.2), turned to 90 degrees
- moved SW2 70.0 mm to (120.3, 106.1)
- moved R11 41.3 mm to (125.3, 85.1), turned to 90 degrees
- moved C8 41.3 mm to (143.2, 96.0), turned to 90 degrees
- moved SW3 30.8 mm to (139.2, 91.1), turned to 45 degrees
- moved C2 7.70 mm to (103.4, 107.7), turned to 0 degrees
- moved R7 1.90 mm to (135.2, 103.8)
- moved D5 1.80 mm to (138.7, 102.0)
- moved D6 1.80 mm to (138.7, 103.7)
- moved R6 1.60 mm to (135.2, 102.0)
- moved C7 0.61 mm to (128.6, 104.9)
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Connections:
- R11 pad 1: /USR_SW -> /PB3-USR_SW
- SW3 pad 2: /USR_SW -> /PB3-USR_SW
Routing:
- net /BOOT0-(DFU): track 0.00 -> 65.3 mm, vias 0 -> 2
- net /PA14-GRN: track 0.00 -> 32.3 mm, vias 0 -> 4
- net Net-(C8-Pad1): track 0.00 -> 26.0 mm, vias 0 -> 2
- net +3V3: track 115.0 -> 138.5 mm
- net /NRST: track 0.00 -> 23.0 mm, vias 0 -> 2
- net /PB3-USR_SW: track 0.00 -> 22.1 mm, vias 0 -> 2
- net /PB4-BLU: track 0.00 -> 19.7 mm
- net /PA15-YEL: track 0.00 -> 17.3 mm
- net /PA13-RED: track 0.00 -> 15.7 mm, vias 0 -> 2
- net Net-(C7-Pad1): track 0.00 -> 8.10 mm
- net +5V: track 129.5 -> 127.0 mm
- net Net-(D5-Pad2): track 0.00 -> 2.12 mm
- net Net-(D6-Pad2): track 0.00 -> 2.03 mm
- net Net-(D4-Pad2): track 0.00 -> 1.97 mm
- net Net-(D7-Pad1): track 0.00 -> 1.92 mm
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- added copper zone on B.Cu, net GND

Commit message: fixed missing envelope out trace
Connections:
- C3 pad 1: /ADC_0 -> /ENVELOPE_OUT
- D1 pad 3: /ADC_0 -> /ENVELOPE_OUT
- R4 pad 2: /ADC_0 -> /ENVELOPE_OUT
- U3 pad 17: Net-(U3-Pad17) -> /ENVELOPE_OUT
Routing:
- net /ENVELOPE_OUT: track 0.00 -> 51.3 mm, vias 0 -> 2
- net /ADC_0: track 12.4 -> 0.00 mm
- net +3V3: track 138.5 -> 132.2 mm
